Commit message: WIP: ros2 control integration

File: src/brunhilde_description/resource/xacro/brunhilde.urdf.xacro (robot description, xacro)
@@ -1,8 +1,4 @@
 <?xml version="1.0" ?>
-<robot name="brunhilde"
-  xmlns:controller="http://playerstage.sourceforge.net/gazebo/xmlschema/#controller"
-  xmlns:interface="http://playerstage.sourceforge.net/gazebo/xmlschema/#interface"
-  xmlns:sensor="http://playerstage.sourceforge.net/gazebo/xmlschema/#sensor"
-  xmlns:xacro="http://playerstage.sourceforge.net/gazebo/xmlschema/#interface">
+<robot name="brunhilde" xmlns:xacro="http://www.ros.org/wiki/xacro">
   <xacro:property name="color_name" value="petrol" />
   <xacro:property name="mesh_ext" value="stl" />
@@ -11,7 +7,9 @@
     <color rgba="0.0 0.59 1.0 1.0"/>
   </material>
-  <xacro:include filename="brunhilde_gazebo.xacro"/>
-  <link name="dummy">
-  </link>
+  <link name="world"/>
+  <joint name="fixed" type="fixed">
+    <parent link="world"/>
+    <child link="base_link"/>
+  </joint>
   <!-- This file is based on: https://atlas.is.localnet/confluence/display/AMDW/Quadruped+URDF+Files -->
   <link name="base_link">
@@ -38,9 +36,4 @@
     </inertial>
   </link>
-  <!-- Dummy joint to connect the base_link to the world -->
-  <joint name="dummy_joint" type="fixed">
-    <parent link="dummy"/>
-    <child link="base_link"/>
-  </joint>
   <xacro:include filename="leg.xacro"/>
   <!-- Include the front left leg -->
@@ -76,3 +69,7 @@
     mesh_ext="${mesh_ext}"
     color_name="${color_name}"/>
+  <xacro:include filename="brunhilde_gazebo.xacro"/>
+  <xacro:property name="use_mock_hardware" value="false"/>
+  <xacro:property name="use_sim_hardware" value="true"/>
+  <xacro:include filename="brunhilde_ros2_control.urdf.xacro"/>
 </robot>

File: src/brunhilde_description/resource/xacro/brunhilde_gazebo.xacro (robot description, xacro)
@@ -1,57 +1,36 @@
 <?xml version="1.0" ?>
-<robot name="brunhilde">
-  <gazebo reference="base_link">
-    <material>Gazebo/Blue</material>
-  </gazebo>
-  <gazebo reference="FL_FOOT">
-    <material>Gazebo/Blue</material>
-  </gazebo>
-  <gazebo reference="FL_LOWER_LEG">
-    <material>Gazebo/Blue</material>
-  </gazebo>
-  <gazebo reference="FL_UPPER_LEG">
-    <material>Gazebo/Blue</material>
-  </gazebo>
-  <gazebo reference="FR_FOOT">
-    <material>Gazebo/Blue</material>
-  </gazebo>
-  <gazebo reference="FR_LOWER_LEG">
-    <material>Gazebo/Blue</material>
-  </gazebo>
-  <gazebo reference="FR_UPPER_LEG">
-    <material>Gazebo/Blue</material>
-  </gazebo>
-  <gazebo reference="HL_FOOT">
-    <material>Gazebo/Blue</material>
-  </gazebo>
-  <gazebo reference="HL_LOWER_LEG">
-    <material>Gazebo/Blue</material>
-  </gazebo>
-  <gazebo reference="HL_UPPER_LEG">
-    <material>Gazebo/Blue</material>
-  </gazebo>
-  <gazebo reference="HR_FOOT">
-    <material>Gazebo/Blue</material>
-  </gazebo>
-  <gazebo reference="HR_LOWER_LEG">
-    <material>Gazebo/Blue</material>
-  </gazebo>
-  <gazebo reference="HR_UPPER_LEG">
-    <material>Gazebo/Blue</material>
-  </gazebo>
-  <gazebo>
-    <plugin name="gazebo_ros_joint_state_publisher"
-            filename="libgazebo_ros_joint_state_publisher.so">
-      <update_rate>20</update_rate>
-      <joint_name>FL_HFE</joint_name>
-      <joint_name>FL_KFE</joint_name>
-      <joint_name>FR_HFE</joint_name>
-      <joint_name>FR_KFE</joint_name>
-      <joint_name>HL_HFE</joint_name>
-      <joint_name>HL_KFE</joint_name>
-      <joint_name>HR_HFE</joint_name>
-      <joint_name>HR_KFE</joint_name>
-      <always_on>true</always_on>
-    </plugin>
-  </gazebo>
+<robot name="brunhilde" xmlns:xacro="http://www.ros.org/wiki/xacro">
+  <xacro:macro name="gz_mat" params="link">
+    <gazebo reference="${link}">
+      <material>
+        <ambient>1 0 0 1</ambient>
+        <diffuse>1 0 0 1</diffuse>
+        <specular>0.1 0.1 0.1 1</specular>
+      </material>
+    </gazebo>
+  </xacro:macro>
+  <xacro:gz_mat link="base_link" />
+  <xacro:gz_mat link="FL_FOOT" />
+  <xacro:gz_mat link="FL_LOWER_LEG" />
+  <xacro:gz_mat link="FL_UPPER_LEG" />
+  <xacro:gz_mat link="FR_FOOT" />
+  <xacro:gz_mat link="FR_LOWER_LEG" />
+  <xacro:gz_mat link="FR_UPPER_LEG" />
+  <xacro:gz_mat link="HL_FOOT" />
+  <xacro:gz_mat link="HL_LOWER_LEG" />
+  <xacro:gz_mat link="HL_UPPER_LEG" />
+  <xacro:gz_mat link="HR_FOOT" />
+  <xacro:gz_mat link="HR_LOWER_LEG" />
+  <xacro:gz_mat link="HR_UPPER_LEG" />
+  <!--<plugin filename="gz-sim-joint-state-publisher-system"
+          name="gz::sim::systems::JointStatePublisher">
+    <joint_name>FL_HFE</joint_name>
+    <joint_name>FL_KFE</joint_name>
+    <joint_name>FR_HFE</joint_name>
+    <joint_name>FR_KFE</joint_name>
+    <joint_name>HL_HFE</joint_name>
+    <joint_name>HL_KFE</joint_name>
+    <joint_name>HR_HFE</joint_name>
+    <joint_name>HR_KFE</joint_name>
+  </plugin>-->
 </robot>

Commit message: updates

File: src/brunhilde_description/resource/xacro/brunhilde.urdf.xacro (robot description, xacro)
@@ -70,6 +70,7 @@
     color_name="${color_name}"/>
   <xacro:include filename="brunhilde_gazebo.xacro"/>
-  <xacro:property name="use_mock_hardware" value="false"/>
-  <xacro:property name="use_sim_hardware" value="true"/>
+  <xacro:property name="use_mock_hardware" value="true"/>
+  <xacro:property name="use_sim_hardware" value="false"/>
+  <xacro:property name="use_real_hardware" value="false"/>
   <xacro:include filename="brunhilde_ros2_control.urdf.xacro"/>
 </robot>

File: src/brunhilde_description/resource/xacro/brunhilde_ros2_control.urdf.xacro (robot description, xacro)
@@ -43,35 +43,35 @@
         		<plugin>gz_ros2_control/GazeboSimSystem</plugin>
 			</xacro:if>
-      <!--<xacro:if value="${use_mock_hardware}">
-        <plugin>mock_components/GenericSystem</plugin>
-        <param name="calculate_dynamics">true</param>
+			<xacro:if value="${use_mock_hardware}">
+				<plugin>mock_components/GenericSystem</plugin>
+				<param name="calculate_dynamics">true</param>
 				<param name="state_following_offset">0.0</param>
-			</xacro:if>-->
-        <xacro:unless value="${use_sim_hardware}">
-          <plugin>ros2_control_odri/SystemOdriHardware</plugin>
-          <property name="prop_config_yaml" value="$(find brunhilde_description)/config/config_solo8.yaml" />
-          <param name="odri_config_yaml">${prop_config_yaml}</param>
-          <param name="desired_starting_position">0.0 0.0 0.0 0.0 0.0 0.0 0.0 0.0</param>
-          <param name="default_joint_cmd">
-            FL_HFE 0.0 0.0 0.0 3.0 0.05
-            FL_KFE 0.0 0.0 0.0 3.0 0.05
-            FR_HFE 0.0 0.0 0.0 3.0 0.05
-            FR_KFE 0.0 0.0 0.0 3.0 0.05
-            HL_HFE 0.0 0.0 0.0 3.0 0.05
-            HL_KFE 0.0 0.0 0.0 3.0 0.05
-            HR_HFE 0.0 0.0 0.0 3.0 0.05
-            HR_KFE 0.0 0.0 0.0 3.0 0.05
-          </param>
-          <param name="default_joint_state">
-            FL_HFE 0.0 0.0 0.0 3.0 0.05
-            FL_KFE 0.0 0.0 0.0 3.0 0.05
-            FR_HFE 0.0 0.0 0.0 3.0 0.05
-            FR_KFE 0.0 0.0 0.0 3.0 0.05
-            HL_HFE 0.0 0.0 0.0 3.0 0.05
-            HL_KFE 0.0 0.0 0.0 3.0 0.05
-            HR_HFE 0.0 0.0 0.0 3.0 0.05
-            HR_KFE 0.0 0.0 0.0 3.0 0.05
-          </param>
-      </xacro:unless>
+			</xacro:if>
+			<xacro:if value="${use_real_hardware}">
+				<plugin>ros2_control_odri/SystemOdriHardware</plugin>
+				<property name="prop_config_yaml" value="$(find brunhilde_description)/config/config_solo8.yaml" />
+				<param name="odri_config_yaml">${prop_config_yaml}</param>
+				<param name="desired_starting_position">0.0 0.0 0.0 0.0 0.0 0.0 0.0 0.0</param>
+				<param name="default_joint_cmd">
+					FL_HFE 0.0 0.0 0.0 3.0 0.05
+					FL_KFE 0.0 0.0 0.0 3.0 0.05
+					FR_HFE 0.0 0.0 0.0 3.0 0.05
+					FR_KFE 0.0 0.0 0.0 3.0 0.05
+					HL_HFE 0.0 0.0 0.0 3.0 0.05
+					HL_KFE 0.0 0.0 0.0 3.0 0.05
+					HR_HFE 0.0 0.0 0.0 3.0 0.05
+					HR_KFE 0.0 0.0 0.0 3.0 0.05
+				</param>
+				<param name="default_joint_state">
+					FL_HFE 0.0 0.0 0.0 3.0 0.05
+					FL_KFE 0.0 0.0 0.0 3.0 0.05
+					FR_HFE 0.0 0.0 0.0 3.0 0.05
+					FR_KFE 0.0 0.0 0.0 3.0 0.05
+					HL_HFE 0.0 0.0 0.0 3.0 0.05
+					HL_KFE 0.0 0.0 0.0 3.0 0.05
+					HR_HFE 0.0 0.0 0.0 3.0 0.05
+					HR_KFE 0.0 0.0 0.0 3.0 0.05
+				</param>
+			</xacro:if>
 		</hardware>
 		<xacro:ros2_control_joint link="FL_HFE" />
@@ -84,11 +84,13 @@
 		<xacro:ros2_control_joint link="HR_KFE" />
 	</ros2_control>
-	<gazebo>
-    <plugin filename="libgz_ros2_control-system.so" name="gz_ros2_control::GazeboSimROS2ControlPlugin">
-		<parameters>$(find brunhilde_control)/config/ros2_control.yaml</parameters>
-		<parameters>$(find brunhilde_control)/config/ros2_control_gz_time.yaml</parameters>
-		<robot_param>robot_description</robot_param>
-      	<robot_param_node>robot_state_publisher</robot_param_node>
-    </plugin>
-	</gazebo>
+	<xacro:if value="${use_sim_hardware}">
+		<gazebo>
+			<plugin filename="libgz_ros2_control-system.so" name="gz_ros2_control::GazeboSimROS2ControlPlugin">
+				<parameters>$(find brunhilde_control)/config/ros2_control.yaml</parameters>
+				<parameters>$(find brunhilde_control)/config/ros2_control_gz_time.yaml</parameters>
+				<robot_param>robot_description</robot_param>
+				<robot_param_node>robot_state_publisher</robot_param_node>
+			</plugin>
+		</gazebo>
+	</xacro:if>
 </robot>

Commit message: first working control example

File: src/brunhilde_description/resource/xacro/brunhilde.urdf.xacro (robot description, xacro)
@@ -70,7 +70,4 @@
     color_name="${color_name}"/>
   <xacro:include filename="brunhilde_gazebo.xacro"/>
-  <xacro:property name="use_mock_hardware" value="true"/>
-  <xacro:property name="use_sim_hardware" value="false"/>
-  <xacro:property name="use_real_hardware" value="false"/>
   <xacro:include filename="brunhilde_ros2_control.urdf.xacro"/>
 </robot>

File: src/brunhilde_description/resource/xacro/brunhilde_ros2_control.urdf.xacro (robot description, xacro)
@@ -1,4 +1,7 @@
 <?xml version="1.0"?>
 <robot name="brunhilde" xmlns:xacro="http://www.ros.org/wiki/xacro">
+  	<xacro:arg name="use_sim_hardware" default="false"/>
+	<xacro:arg name="use_mock_hardware" default="false"/>
+	<xacro:arg name="use_real_hardware" default="true"/>
 	<ros2_control name="brunhilde" type="system">
     <xacro:macro name="ros2_control_joint" params="link">
@@ -40,15 +43,14 @@
 		</xacro:macro>
 		<hardware>
-			<xacro:if value="${use_sim_hardware}">
+			<xacro:if value="$(arg use_sim_hardware)">
         		<plugin>gz_ros2_control/GazeboSimSystem</plugin>
 			</xacro:if>
-			<xacro:if value="${use_mock_hardware}">
+			<xacro:if value="$(arg use_mock_hardware)">
 				<plugin>mock_components/GenericSystem</plugin>
-				<param name="calculate_dynamics">true</param>
 				<param name="state_following_offset">0.0</param>
 			</xacro:if>
-			<xacro:if value="${use_real_hardware}">
+			<xacro:if value="$(arg use_real_hardware)">
 				<plugin>ros2_control_odri/SystemOdriHardware</plugin>
-				<property name="prop_config_yaml" value="$(find brunhilde_description)/config/config_solo8.yaml" />
+				<xacro:property name="prop_config_yaml" value="$(find brunhilde_description)/config/config_solo8.yaml" />
 				<param name="odri_config_yaml">${prop_config_yaml}</param>
 				<param name="desired_starting_position">0.0 0.0 0.0 0.0 0.0 0.0 0.0 0.0</param>
@@ -84,5 +86,5 @@
 		<xacro:ros2_control_joint link="HR_KFE" />
 	</ros2_control>
-	<xacro:if value="${use_sim_hardware}">
+	<xacro:if value="$(arg use_sim_hardware)">
 		<gazebo>
 			<plugin filename="libgz_ros2_control-system.so" name="gz_ros2_control::GazeboSimROS2ControlPlugin">

Commit message: gz sim integration

File: src/brunhilde_description/resource/xacro/brunhilde.urdf.xacro (robot description, xacro)
@@ -7,11 +7,13 @@
     <color rgba="0.0 0.59 1.0 1.0"/>
   </material>
-  <link name="world"/>
-  <joint name="fixed" type="fixed">
-    <parent link="world"/>
-    <child link="base_link"/>
+  <link name="base_link">
+  </link>
+  <joint name="base_joint" type="fixed">
+    <origin xyz="0 0 0" rpy="0 0 0" />
+    <parent link="base_link"/>
+    <child link="body_frame"/>
   </joint>
   <!-- This file is based on: https://atlas.is.localnet/confluence/display/AMDW/Quadruped+URDF+Files -->
-  <link name="base_link">
+  <link name="body_frame">
     <visual>
       <origin xyz="0 0 0" rpy="0 0 0" />

File: src/brunhilde_description/resource/xacro/leg.xacro (robot description, xacro)
@@ -18,5 +18,5 @@
     <!-- Joint between the base and the ${prefix} upper leg -->
     <joint name="${prefix}_HFE" type="revolute">
-      <parent link="base_link"/>
+      <parent link="body_frame"/>
       <child link="${prefix}_UPPER_LEG"/>
       <limit effort="1000" lower="-10" upper="10" velocity="1000"/>

Commit message: new collision model

File: src/brunhilde_description/resource/xacro/brunhilde.urdf.xacro (robot description, xacro)
@@ -4,4 +4,5 @@
   <xacro:property name="mesh_ext" value="stl" />
   <xacro:property name="mesh_path" value="package://brunhilde_description/resource/xacro/meshes/" />
+  <xacro:property name="col_mesh_path" value="package://brunhilde_description/resource/xacro/collisions/" />
   <material name="${color_name}">
     <color rgba="0.0 0.59 1.0 1.0"/>
@@ -26,5 +27,5 @@
       <origin xyz="0 0 0" rpy="0 0 0" />
       <geometry>
-        <mesh filename="${mesh_path}solo_body.${mesh_ext}"/>
+        <mesh filename="${col_mesh_path}solo_body.${mesh_ext}"/>
       </geometry>
     </collision>
@@ -46,4 +47,5 @@
     mesh_path="${mesh_path}"
     mesh_ext="${mesh_ext}"
+    col_mesh_path="${col_mesh_path}"
     color_name="${color_name}"/>
   <!-- Include the front right leg -->
@@ -54,4 +56,5 @@
     mesh_path="${mesh_path}"
     mesh_ext="${mesh_ext}"
+    col_mesh_path="${col_mesh_path}"
     color_name="${color_name}"/>
   <!-- Include the hind left leg -->
@@ -62,4 +65,5 @@
     mesh_path="${mesh_path}"
     mesh_ext="${mesh_ext}"
+    col_mesh_path="${col_mesh_path}"
     color_name="${color_name}"/>
   <!-- Include the hind right leg -->
@@ -70,4 +74,5 @@
     mesh_path="${mesh_path}"
     mesh_ext="${mesh_ext}"
+    col_mesh_path="${col_mesh_path}"
     color_name="${color_name}"/>
   <xacro:include filename="brunhilde_gazebo.xacro"/>

File: src/brunhilde_description/resource/xacro/leg.xacro (robot description, xacro)
@@ -15,5 +15,5 @@
   <!-- Macro defining solo leg. -->
   <xacro:macro name="leg" params="prefix is_front is_right mesh_path
-                                  mesh_ext color_name">
+                                  mesh_ext col_mesh_path color_name">
     <!-- Joint between the base and the ${prefix} upper leg -->
     <joint name="${prefix}_HFE" type="revolute">
@@ -83,8 +83,8 @@
         <geometry>
           <xacro:unless value="${is_right}">
-            <mesh filename="${mesh_path}solo_upper_leg_left_side.${mesh_ext}"/>
+            <mesh filename="${col_mesh_path}solo_upper_leg_left_side.${mesh_ext}"/>
           </xacro:unless>
           <xacro:if value="${is_right}">
-            <mesh filename="${mesh_path}solo_upper_leg_right_side.${mesh_ext}"/>
+            <mesh filename="${col_mesh_path}solo_upper_leg_right_side.${mesh_ext}"/>
           </xacro:if>
         </geometry>
@@ -160,8 +160,8 @@
         <geometry>
           <xacro:unless value="${is_right}">
-            <mesh filename="${mesh_path}solo_lower_leg_v2_left_side.${mesh_ext}"/>
+            <mesh filename="${col_mesh_path}solo_lower_leg_v2_left_side.${mesh_ext}"/>
           </xacro:unless>
           <xacro:if value="${is_right}">
-            <mesh filename="${mesh_path}solo_lower_leg_v2_right_side.${mesh_ext}"/>
+            <mesh filename="${col_mesh_path}solo_lower_leg_v2_right_side.${mesh_ext}"/>
           </xacro:if>
         </geometry>
