Commit message: Port to watschel complete

File: src/watschel_description/resource/xacro/example_robot.urdf.xacro (robot description, xacro)
@@ -23,5 +23,5 @@
         <visual>
             <geometry>
-                <mesh filename="package://watschel_urdf_creation/meshes/3d_modelle/Hip.stl" scale="0.01 0.01 0.01"/>
+                <mesh filename="package://watschel_description/meshes/3d_modelle/Hip.stl" scale="0.01 0.01 0.01"/>
             </geometry>
             <material name="green">
@@ -51,5 +51,5 @@
         <visual>
             <geometry>
-                <mesh filename="package://watschel_urdf_creation/meshes/3d_modelle/Left_leg/Top_leg_front.stl" scale="0.01 0.01 0.01"/>
+                <mesh filename="package://watschel_description/meshes/3d_modelle/Left_leg/Top_leg_front.stl" scale="0.01 0.01 0.01"/>
             </geometry>
             <material name="green">
@@ -87,5 +87,6 @@
         <visual>
             <geometry>
-                <mesh filename="package://watschel_urdf_creation/meshes/3d_modelle/Right_leg/Top_leg_front.stl" scale="0.01 0.01 0.01"/>
+                <mesh filename="package://watschel_description/meshes/3d_modelle/Right_leg/Top_leg_front.stl" scale="0.01 0.01 0.01"/>
+                <box size="0.6 0.1 0.2"/>
             </geometry>
             <material name="green">
@@ -105,5 +106,5 @@
         <visual>
             <geometry>
-                <mesh filename="package://watschel_urdf_creation/meshes/3d_modelle/Left_leg/Knee.stl" scale="0.01 0.01 0.01"/>
+                <mesh filename="package://watschel_description/meshes/3d_modelle/Left_leg/Knee.stl" scale="0.01 0.01 0.01"/>
             </geometry>
             <material name="green">
@@ -123,5 +124,5 @@
         <visual>
             <geometry>
-                <mesh filename="package://watschel_urdf_creation/meshes/3d_modelle/Left_leg/Knee.stl" scale="0.01 0.01 0.01"/>
+                <mesh filename="package://watschel_description/meshes/3d_modelle/Left_leg/Knee.stl" scale="0.01 0.01 0.01"/>
             </geometry>
             <material name="green">
@@ -140,5 +141,5 @@
         <visual>
             <geometry>
-                <mesh filename="package://watschel_urdf_creation/meshes/3d_modelle/Right_leg/Low_leg_front.stl" scale="0.01 0.01 0.01"/>
+                <mesh filename="package://watschel_description/meshes/3d_modelle/Right_leg/Low_leg_front.stl" scale="0.01 0.01 0.01"/>
             </geometry>
             <material name="green">
@@ -157,5 +158,5 @@
         <visual>
             <geometry>
-                <mesh filename="package://watschel_urdf_creation/meshes/3d_modelle/Left_leg/Low_leg_front.stl" scale="0.01 0.01 0.01"/>
+                <mesh filename="package://watschel_description/meshes/3d_modelle/Left_leg/Low_leg_front.stl" scale="0.01 0.01 0.01"/>
             </geometry>
             <material name="green">
@@ -175,5 +176,5 @@
         <visual>
             <geometry>
-                <mesh filename="package://watschel_urdf_creation/meshes/3d_modelle/Left_leg/Foot.stl" scale="0.01 0.01 0.01"/>
+                <mesh filename="package://watschel_description/meshes/3d_modelle/Left_leg/Foot.stl" scale="0.01 0.01 0.01"/>
             </geometry>
             <material name="green">
@@ -193,5 +194,5 @@
         <visual>
             <geometry>
-                <mesh filename="package://watschel_urdf_creation/meshes/3d_modelle/Left_leg/Foot.stl" scale="0.01 0.01 0.01"/>
+                <mesh filename="package://watschel_description/meshes/3d_modelle/Left_leg/Foot.stl" scale="0.01 0.01 0.01"/>
             </geometry>
             <material name="green">

Commit message: Watschel now living in gazebo

File: src/watschel_description/resource/xacro/example_robot.urdf.xacro (robot description, xacro)
@@ -6,13 +6,4 @@
     <xacro:property name="joint_angle" value="${pi/4}" />
     <xacro:property name="knee_angle" value="joint_angle*2" />
-    <!-- This first link called "world" is empty -->
-    <link name="world"></link>
-    <!-- A simple fixed joint from our empty world link, to our base. -->
-    <!-- The base origin is offset from the world origin. -->
-    <joint name="base_joint" type="fixed">
-        <origin xyz="0 0 1" rpy="0 0 0"/>
-        <parent link="world"/>
-        <child link="base_link"/>
-    </joint>
     <!-- base_link is a large rectangular plate. Some things to note: -->
     <!-- - We set the visual origin Z to half the box height, so that the link origin sits at the bottom of the box -->
@@ -29,10 +20,4 @@
             </material>
         </visual>
-        <collision>
-            <origin xyz="0 0 0.0" rpy="0 0 0"/>
-            <geometry>
-                <box size="7 3 0.1" />
-            </geometry>
-        </collision>
         <inertial>
             <origin xyz="0 0 0.05" rpy="0 0 0"/>
@@ -57,4 +42,8 @@
             </material>
         </visual>
+        <inertial>
+            <mass value="10"/>
+            <inertia ixx="0.4" ixy="0.0" ixz="0.0" iyy="0.4" iyz="0.0" izz="0.2"/>
+        </inertial>
     </link>
     <joint name="support_upper_left_joint" type="revolute">
@@ -67,13 +56,8 @@
     </joint>
     <link name="support_upper_left">
-        <visual>
-            <geometry>
-                <cylinder length="0.6" radius="0.07"/>
-                <origin xyz="0 0 -0.6"/>
-            </geometry>
-            <material name="green">
-                <color rgba="0.2 1 0.2 1"/>
-            </material>
-        </visual>
+        <inertial>
+            <mass value="10"/>
+            <inertia ixx="0.4" ixy="0.0" ixz="0.0" iyy="0.4" iyz="0.0" izz="0.2"/>
+        </inertial>
     </link>
     <joint name="right_hip_joint" type="revolute">
@@ -94,4 +78,8 @@
             </material>
         </visual>
+        <inertial>
+            <mass value="10"/>
+            <inertia ixx="0.4" ixy="0.0" ixz="0.0" iyy="0.4" iyz="0.0" izz="0.2"/>
+        </inertial>
     </link>
     <joint name="knee_left_joint" type="revolute">
@@ -112,4 +100,8 @@
             </material>
         </visual>
+        <inertial>
+            <mass value="10"/>
+            <inertia ixx="0.4" ixy="0.0" ixz="0.0" iyy="0.4" iyz="0.0" izz="0.2"/>
+        </inertial>
     </link>
     <joint name="knee_right_joint" type="revolute">
@@ -130,4 +122,8 @@
             </material>
         </visual>
+        <inertial>
+            <mass value="10"/>
+            <inertia ixx="0.4" ixy="0.0" ixz="0.0" iyy="0.4" iyz="0.0" izz="0.2"/>
+        </inertial>
     </link>
     <joint name="lower_leg_right_joint" type="revolute">
@@ -147,4 +143,8 @@
             </material>
         </visual>
+        <inertial>
+            <mass value="10"/>
+            <inertia ixx="0.4" ixy="0.0" ixz="0.0" iyy="0.4" iyz="0.0" izz="0.2"/>
+        </inertial>
     </link>
     <joint name="lower_leg_left_joint" type="revolute">
@@ -164,4 +164,8 @@
             </material>
         </visual>
+        <inertial>
+            <mass value="10"/>
+            <inertia ixx="0.4" ixy="0.0" ixz="0.0" iyy="0.4" iyz="0.0" izz="0.2"/>
+        </inertial>
     </link>
     <joint name="foot_left_joint" type="revolute">
@@ -182,4 +186,13 @@
             </material>
         </visual>
+        <collision>
+            <geometry>
+                <box size="0.2 0.2 0.1"/>
+            </geometry>
+        </collision>
+        <inertial>
+            <mass value="10"/>
+            <inertia ixx="0.4" ixy="0.0" ixz="0.0" iyy="0.4" iyz="0.0" izz="0.2"/>
+        </inertial>
     </link>
     <joint name="foot_right_joint" type="revolute">
@@ -200,5 +213,15 @@
             </material>
         </visual>
+        <collision>
+            <geometry>
+                <box size="0.2 0.2 0.1"/>
+            </geometry>
+        </collision>
+        <inertial>
+            <mass value="10"/>
+            <inertia ixx="0.4" ixy="0.0" ixz="0.0" iyy="0.4" iyz="0.0" izz="0.2"/>
+        </inertial>
     </link>
     <!--xacro:include filename="example_gazebo.xacro" /-->
+    <xacro:include filename="watschel_ros2_control.urdf.xacro"/>
 </robot>

Commit message: change physx engine

File: src/watschel_description/resource/xacro/example_robot.urdf.xacro (robot description, xacro)
@@ -188,5 +188,5 @@
         <collision>
             <geometry>
-                <box size="0.2 0.2 0.1"/>
+                <box size="0.4 0.8 0.1"/>
             </geometry>
         </collision>
@@ -215,5 +215,5 @@
         <collision>
             <geometry>
-                <box size="0.2 0.2 0.1"/>
+                <box size="0.4 0.8 0.1"/>
             </geometry>
         </collision>

File: src/watschel_description/resource/xacro/watschel_ros2_control_mimics.xacro (robot description, xacro)
@@ -4,30 +4,11 @@
 	<xacro:arg name="use_mock_hardware" default="false"/>
 	<xacro:arg name="use_real_hardware" default="false"/>
-	<ros2_control name="watschel" type="system">
-    <xacro:macro name="ros2_control_joint" params="link">
+	<ros2_control name="watschel_mimics" type="system">
+    <xacro:macro name="ros2_control_joint" params="link mimic">
 			<joint name="${link}">
-				<command_interface name="position">
-					<param name="min">-0.5</param>
-					<param name="max">0.5</param>
-				</command_interface>
-				<command_interface name="velocity">
-					<param name="min">-1</param>
-					<param name="max">1</param>
-				</command_interface>
-				<command_interface name="effort">
-					<param name="min">-1</param>
-					<param name="max">1</param>
-				</command_interface>
 				<state_interface name="position" />
 				<state_interface name="velocity" />
 				<state_interface name="effort" />
-				<param name="motor_number">0</param>
-				<param name="gear_ratio">9.</param>
-				<param name="motor_constant">0.025</param>
-				<param name="max_current">12.</param>
-				<param name="maxObject_joint_velocity">80.</param>
-				<param name="safety_damping">0.5</param>
-				<param name="motor_reversed_polarity">true</param>
-				<param name="position_offset">0.238</param>
+				<mimic joint="${mimic}" multiplier="1" offset="0"></mimic>
 			</joint>
 		</xacro:macro>
@@ -59,8 +40,5 @@
 			</xacro:if>
 		</hardware>
-		<xacro:ros2_control_joint link="left_hip_joint" />
-		<xacro:ros2_control_joint link="right_hip_joint" />
-		<xacro:ros2_control_joint link="lower_leg_right_joint" />
-		<xacro:ros2_control_joint link="lower_leg_left_joint" />
+		<xacro:ros2_control_joint link="foot_left_joint" mimic="left_knee_joint"/>
 	</ros2_control>
 	<xacro:if value="$(arg use_sim_hardware)">

Commit message: Watschel sim now worksgit add .!

File: src/watschel_description/resource/xacro/example_robot.urdf.xacro (robot description, xacro)
@@ -4,12 +4,19 @@
     <!-- As we move through the file, new things to note will be pointed out. -->
     <!-- It's not meant an example of GOOD design, but an example of some of the various features of URDF/xacro. -->
+    <link name="base_link">
+    </link>
+    <joint name="base_joint" type="fixed">
+      <origin xyz="0 0 0" rpy="0 0 0" />
+      <parent link="base_link"/>
+      <child link="body_frame"/>
+    </joint>
     <xacro:property name="joint_angle" value="${pi/4}" />
     <xacro:property name="knee_angle" value="joint_angle*2" />
-    <!-- base_link is a large rectangular plate. Some things to note: -->
+    <!-- body_frame is a large rectangular plate. Some things to note: -->
     <!-- - We set the visual origin Z to half the box height, so that the link origin sits at the bottom of the box -->
     <!-- - We set the collision to be identical to the visual -->
     <!-- - We specified the colour manually (but still need to enter a name) -->
     <!-- - We specified all the inertial parameters manually -->
-    <link name="base_link">
+    <link name="body_frame">
         <visual>
             <geometry>
@@ -20,4 +27,11 @@
             </material>
         </visual>
+        <collision>
+            <geometry>
+                <box size="1.2 0.3 0.1">
+                </box>
+                <origin xyz="0.0 4.0 0.0"/>
+            </geometry>
+        </collision>
         <inertial>
             <origin xyz="0 0 0.05" rpy="0 0 0"/>
@@ -28,5 +42,5 @@
     <joint name="left_hip_joint" type="revolute">
         <origin xyz="-0.36 0.24 0.05" rpy="0 0 0"/>
-        <parent link="base_link"/>
+        <parent link="body_frame"/>
         <child link="leg_upper_left"/>
         <axis xyz="-1 0 0"/>
@@ -49,5 +63,5 @@
     <joint name="support_upper_left_joint" type="revolute">
         <origin xyz="-0.36 0.5 0.05" rpy="0 0 0"/>
-        <parent link="base_link"/>
+        <parent link="body_frame"/>
         <child link="support_upper_left"/>
         <axis xyz="-1 0 0"/>
@@ -63,5 +77,5 @@
     <joint name="right_hip_joint" type="revolute">
         <origin xyz="0.36 0.24 0.05" rpy="0 0 0"/>
-        <parent link="base_link"/>
+        <parent link="body_frame"/>
         <child link="leg_upper_right"/>
         <axis xyz="-1 0 0"/>
@@ -83,10 +97,9 @@
         </inertial>
     </link>
-    <joint name="knee_left_joint" type="revolute">
+    <joint name="knee_left_joint" type="fixed">
         <origin xyz="0 0 -0.65" rpy="0 0 0"/>
         <parent link="leg_upper_left"/>
         <child link="knee_left"/>
         <axis xyz="-1 0 0"/>
-        <limit lower="${-pi/4}" upper="${pi/4}" velocity="100" effort="100"/>
         <mimic joint="left_hip_joint" multiplier="-1"/>
     </joint>
@@ -105,10 +118,9 @@
         </inertial>
     </link>
-    <joint name="knee_right_joint" type="revolute">
+    <joint name="knee_right_joint" type="fixed">
         <origin xyz="0 0 -0.65" rpy="0 0 0"/>
         <parent link="leg_upper_right"/>
         <child link="knee_right"/>
         <axis xyz="-1 0 0"/>
-        <limit lower="${-pi/4}" upper="${pi/4}" velocity="100" effort="100"/>
         <mimic joint="right_hip_joint" multiplier="-1"/>
     </joint>
@@ -169,10 +181,9 @@
         </inertial>
     </link>
-    <joint name="foot_left_joint" type="revolute">
+    <joint name="foot_left_joint" type="fixed">
         <origin xyz="0 0.05 -0.65"/>
         <parent link="leg_lower_left"/>
         <child link="foot_left"/>
         <axis xyz="-1 0 0"/>
-        <limit lower="${-pi/4}" upper="${pi/4}" velocity="100" effort="100"/>
         <mimic  joint="lower_leg_left_joint" multiplier="-1" />
     </joint>
@@ -196,10 +207,9 @@
         </inertial>
     </link>
-    <joint name="foot_right_joint" type="revolute">
+    <joint name="foot_right_joint" type="fixed">
         <origin xyz="0 0.05 -0.65"/>
         <parent link="leg_lower_right"/>
         <child link="foot_right"/>
         <axis xyz="-1 0 0"/>
-        <limit lower="${-pi/4}" upper="${pi/4}" velocity="100" effort="100"/>
         <mimic  joint="lower_leg_right_joint" multiplier="-1" />
     </joint>

Commit message: New changes and fix urdf

File: src/watschel_description/resource/xacro/example_robot.urdf.xacro (robot description, xacro)
@@ -36,6 +36,6 @@
         <inertial>
             <origin xyz="0 0 0.05" rpy="0 0 0"/>
-            <mass value="12" />
-            <inertia ixx="2.26" ixy="0.0" ixz="0.0" iyy="6.26" iyz="0.0" izz="8.5" />
+            <mass value="172" />
+            <inertia ixx="65.06899629082241" ixy="0.0" ixz="0.0" iyy="188.99729683407716" iyz="0.0" izz="242.36785108586454" />
         </inertial>
     </link>
@@ -58,5 +58,5 @@
         <inertial>
             <mass value="10"/>
-            <inertia ixx="0.4" ixy="0.0" ixz="0.0" iyy="0.4" iyz="0.0" izz="0.2"/>
+            <inertia ixx="42.70110889206565" ixy="0.0" ixz="0.0" iyy="54.35021715917743" iyz="0.0" izz="15.553565591531272"/>
         </inertial>
     </link>
@@ -94,5 +94,5 @@
         <inertial>
             <mass value="10"/>
-            <inertia ixx="0.4" ixy="0.0" ixz="0.0" iyy="0.4" iyz="0.0" izz="0.2"/>
+            <inertia ixx="42.70110889206565" ixy="0.0" ixz="0.0" iyy="54.35021715917743" iyz="0.0" izz="15.553565591531272"/>
         </inertial>
     </link>
@@ -114,6 +114,6 @@
         </visual>
         <inertial>
-            <mass value="10"/>
-            <inertia ixx="0.4" ixy="0.0" ixz="0.0" iyy="0.4" iyz="0.0" izz="0.2"/>
+            <mass value="20"/>
+            <inertia ixx="50.868164916992344" ixy="0.0" ixz="0.0" iyy="22.91604242324853" iyz="0.0" izz="63.92287750625619"/>
         </inertial>
     </link>
@@ -135,6 +135,6 @@
         </visual>
         <inertial>
-            <mass value="10"/>
-            <inertia ixx="0.4" ixy="0.0" ixz="0.0" iyy="0.4" iyz="0.0" izz="0.2"/>
+            <mass value="20"/>
+            <inertia ixx="50.868164916992344" ixy="0.0" ixz="0.0" iyy="22.91604242324853" iyz="0.0" izz="63.92287750625619"/>
         </inertial>
     </link>
@@ -157,5 +157,5 @@
         <inertial>
             <mass value="10"/>
-            <inertia ixx="0.4" ixy="0.0" ixz="0.0" iyy="0.4" iyz="0.0" izz="0.2"/>
+            <inertia ixx="44.06199538400554" ixy="0.0" ixz="0.0" iyy="60.37315620362157" iyz="0.0" izz="20.349008232508035"/>
         </inertial>
     </link>
@@ -178,5 +178,5 @@
         <inertial>
             <mass value="10"/>
-            <inertia ixx="0.4" ixy="0.0" ixz="0.0" iyy="0.4" iyz="0.0" izz="0.2"/>
+            <inertia ixx="44.06199538400554" ixy="0.0" ixz="0.0" iyy="60.37315620362157" iyz="0.0" izz="20.349008232508035"/>
         </inertial>
     </link>
@@ -203,6 +203,6 @@
         </collision>
         <inertial>
-            <mass value="10"/>
-            <inertia ixx="0.4" ixy="0.0" ixz="0.0" iyy="0.4" iyz="0.0" izz="0.2"/>
+            <mass value="11"/>
+            <inertia ixx="30.922726715508456" ixy="0.0" ixz="0.0" iyy="11.747663442495953" iyz="0.0" izz="31.94689382554976"/>
         </inertial>
     </link>
@@ -217,5 +217,5 @@
         <visual>
             <geometry>
-                <mesh filename="package://watschel_description/meshes/3d_modelle/Left_leg/Foot.stl" scale="0.01 0.01 0.01"/>
+                <mesh filename="package://watschel_description/meshes/3d_modelle/Right_leg/Foot.stl" scale="0.01 0.01 0.01"/>
             </geometry>
             <material name="green">
@@ -229,6 +229,6 @@
         </collision>
         <inertial>
-            <mass value="10"/>
-            <inertia ixx="0.4" ixy="0.0" ixz="0.0" iyy="0.4" iyz="0.0" izz="0.2"/>
+            <mass value="11"/>
+            <inertia ixx="30.922726715508456" ixy="0.0" ixz="0.0" iyy="11.747663442495953" iyz="0.0" izz="31.94689382554976"/>
         </inertial>
     </link>
