Commit message: Many changes which are good for everyone

File: src/watschel_description/resource/xacro/example_robot.urdf.xacro (robot description, xacro)
@@ -35,5 +35,5 @@
         </collision>
         <inertial>
-            <origin xyz="0 0 0.05" rpy="0 0 0"/>
+            <origin xyz="0 0.28 0.09" rpy="0 0 0"/>
             <mass value="172" />
             <inertia ixx="65.06899629082241" ixy="0.0" ixz="0.0" iyy="188.99729683407716" iyz="0.0" izz="242.36785108586454" />
@@ -61,5 +61,5 @@
         </inertial>
     </link>
-    <joint name="support_upper_left_joint" type="revolute">
+    <joint name="support_upper_left_joint" type="fixed">
         <origin xyz="-0.36 0.5 0.05" rpy="0 0 0"/>
         <parent link="body_frame"/>
@@ -67,7 +67,37 @@
         <axis xyz="-1 0 0"/>
         <limit lower="${-pi/4}" upper="${pi/4}" velocity="100" effort="100"/>
-        <mimic joint="left_hip_joint"/>
+        <mimic joint="left_hip_joint" multiplier="1"/>
     </joint>
     <link name="support_upper_left">
+        <visual>
+            <geometry>
+                <mesh filename="package://watschel_description/meshes/3d_modelle/Left_leg/Top_leg_back.stl" scale="0.01 0.01 0.01"/>
+            </geometry>
+            <material name="green">
+                <color rgba="0.2 1 0.2 1"/>
+            </material>
+        </visual>
+        <inertial>
+            <mass value="10"/>
+            <inertia ixx="0.4" ixy="0.0" ixz="0.0" iyy="0.4" iyz="0.0" izz="0.2"/>
+        </inertial>
+    </link>
+    <joint name="support_upper_right_joint" type="fixed">
+        <origin xyz="0.36 0.5 0.05" rpy="0 0 0"/>
+        <parent link="body_frame"/>
+        <child link="support_upper_right"/>
+        <axis xyz="-1 0 0"/>
+        <limit lower="${-pi/4}" upper="${pi/4}" velocity="100" effort="100"/>
+        <mimic joint="left_hip_joint" multiplier="1"/>
+    </joint>
+    <link name="support_upper_right">
+        <visual>
+            <geometry>
+                <mesh filename="package://watschel_description/meshes/3d_modelle/Right_leg/Top_leg_back.stl" scale="0.01 0.01 0.01"/>
+            </geometry>
+            <material name="green">
+                <color rgba="0.2 1 0.2 1"/>
+            </material>
+        </visual>
         <inertial>
             <mass value="10"/>
@@ -97,9 +127,10 @@
         </inertial>
     </link>
-    <joint name="knee_left_joint" type="fixed">
+    <joint name="knee_left_joint" type="revolute">
         <origin xyz="0 0 -0.65" rpy="0 0 0"/>
         <parent link="leg_upper_left"/>
         <child link="knee_left"/>
         <axis xyz="-1 0 0"/>
+        <limit lower="-1" upper="1" effort="0.0" velocity="0.0"/>
         <mimic joint="left_hip_joint" multiplier="-1"/>
     </joint>
@@ -188,4 +219,48 @@
         <mimic  joint="lower_leg_left_joint" multiplier="-1" />
     </joint>
+    <joint name="support_lower_right_joint" type="fixed">
+        <origin xyz="-0.15 0.15 0" rpy="0 0 0"/>
+        <parent link="knee_right"/>
+        <child link="support_lower_right"/>
+        <axis xyz="-1 0 0"/>
+        <limit lower="${-pi/4}" upper="${pi/4}" velocity="100" effort="100"/>
+        <mimic joint="lower_leg_right_joint" multiplier="1"/>
+    </joint>
+    <link name="support_lower_right">
+        <visual>
+            <geometry>
+                <mesh filename="package://watschel_description/meshes/3d_modelle/Right_leg/Low_leg_back.stl" scale="0.01 0.01 0.01"/>
+            </geometry>
+            <material name="green">
+                <color rgba="0.2 1 0.2 1"/>
+            </material>
+        </visual>
+        <inertial>
+            <mass value="10"/>
+            <inertia ixx="0.4" ixy="0.0" ixz="0.0" iyy="0.4" iyz="0.0" izz="0.2"/>
+        </inertial>
+    </link>
+    <joint name="support_lower_left_joint" type="fixed">
+        <origin xyz="0 0.15 0" rpy="0 0 0"/>
+        <parent link="knee_left"/>
+        <child link="support_lower_left"/>
+        <axis xyz="-1 0 0"/>
+        <limit lower="${-pi/4}" upper="${pi/4}" velocity="100" effort="100"/>
+        <mimic joint="lower_leg_left_joint" multiplier="1"/>
+    </joint>
+    <link name="support_lower_left">
+        <visual>
+            <geometry>
+                <mesh filename="package://watschel_description/meshes/3d_modelle/Left_leg/Low_leg_back.stl" scale="0.01 0.01 0.01"/>
+            </geometry>
+            <material name="green">
+                <color rgba="0.2 1 0.2 1"/>
+            </material>
+        </visual>
+        <inertial>
+            <mass value="10"/>
+            <inertia ixx="0.4" ixy="0.0" ixz="0.0" iyy="0.4" iyz="0.0" izz="0.2"/>
+        </inertial>
+    </link>
     <link name="foot_left">
         <visual>

File: src/watschel_description/resource/xacro/watschel_ros2_control.urdf.xacro (robot description, xacro)
@@ -27,5 +27,5 @@
 				<param name="max_current">12.</param>
 				<param name="maxObject_joint_velocity">80.</param>
-				<param name="safety_damping">0.5</param>
+				<param name="safety_damping">0.2</param>
 				<param name="motor_reversed_polarity">true</param>
 				<param name="position_offset">0.238</param>
@@ -44,5 +44,5 @@
 				<xacro:property name="prop_config_yaml" value="$(find watschel_description)/config/config_solo8.yaml" />
 				<param name="odri_config_yaml">${prop_config_yaml}</param>
-				<param name="desired_starting_position">0.0 0.0 0.0 0.0 0.0 0.0 0.0 0.0</param>
+				<param name="desired_starting_position">0.0 0.0 0.0 0.0</param>
 				<param name="default_joint_cmd">
 					left_hip_joint 0.0 0.0 0.0 3.0 0.05
